Commit message: Project 4: update config files

File: Project4/catkin_ws/src/my_robot/urdf/my_robot.xacro (robot description, xacro)
@@ -126,5 +126,5 @@
     <dynamics damping="1.0" friction="1.0"/>
   </joint>
-  <link name="camera">
+  <link name="camera_link">
     <visual name="camera_visual">
       <origin xyz="0 0 0" rpy="0 0 0" />
@@ -155,7 +155,14 @@
     <axis xyz="0 1 0"/>
     <origin xyz="0.3 0 0" rpy="0 0 0" />
-    <child link="camera" />
+    <child link="camera_link" />
     <parent link="chassis" />
   </joint>
+  <joint name="camera_optical_joint" type="fixed">
+    <origin xyz="0 0 0" rpy="-1.5707 0 -1.5707"/>
+    <parent link="camera_link"/>
+    <child link="camera_link_optical"/>
+  </joint>
+  <link name="camera_link_optical">
+  </link>
   <link name="hokuyo">
     <visual name="hokuyo_visual">

Commit message: Project 4: Map My World - complete
Updated all config files and drove around my world. RTabMap was able to generate many loop closures.

File: Project4/catkin_ws/src/my_robot/urdf/my_robot.xacro (robot description, xacro)
@@ -126,5 +126,5 @@
     <dynamics damping="1.0" friction="1.0"/>
   </joint>
-  <link name="camera_link">
+  <link name="camera">
     <visual name="camera_visual">
       <origin xyz="0 0 0" rpy="0 0 0" />
@@ -155,10 +155,10 @@
     <axis xyz="0 1 0"/>
     <origin xyz="0.3 0 0" rpy="0 0 0" />
-    <child link="camera_link" />
+    <child link="camera" />
     <parent link="chassis" />
   </joint>
   <joint name="camera_optical_joint" type="fixed">
     <origin xyz="0 0 0" rpy="-1.5707 0 -1.5707"/>
-    <parent link="camera_link"/>
+    <parent link="camera"/>
     <child link="camera_link_optical"/>
   </joint>

Commit message: Project 4: Fix teleop robot control and rtabmap.db
Problem was the caster wheels. I removed one and fixed the joint and friction for the other.

Also updated the rtabmap with a cleaner version.

File: Project4/catkin_ws/src/my_robot/urdf/my_robot.xacro (robot description, xacro)
@@ -33,32 +33,28 @@
       />
     </inertial>
-    <visual name='back_caster_visual'>
-      <origin xyz="-0.2 0 -0.1" rpy=" 0 0 0"/>
+  </link>
+  <link name="caster_wheel">
+    <visual>
       <geometry>
         <sphere radius="0.1"/>
       </geometry>
     </visual>
-    <collision name='back_caster_collision'>
-      <origin xyz="-0.2 0 -0.1" rpy=" 0 0 0"/>
+    <collision>
       <geometry>
         <sphere radius="0.0999"/>
       </geometry>
     </collision>
-    <visual name='front_caster_visual'>
-      <origin xyz="0.2 0 -0.1" rpy=" 0 0 0"/>
-      <geometry>
-        <sphere radius="0.1"/>
-      </geometry>
-    </visual>
-    <collision name='front_caster_collision'>
-      <origin xyz="0.2 0 -0.1" rpy=" 0 0 0"/>
-      <geometry>
-        <sphere radius="0.0999"/>
-      </geometry>
-    </collision>
+    <inertial>
+      <mass value="0.1"/>
+      <origin xyz="0 0 0" rpy=" 0 0 0"/>
+      <inertia
+          ixx="0.1" ixy="0" ixz="0"
+          iyy="0.1" iyz="0"
+          izz="0.1"
+      />
+    </inertial>
   </link>
   <link name="left_wheel">
     <visual name="left_wheel_visual">
-      <origin xyz="0 0.11 0" rpy=" 0 1.5707 1.5707"/>
       <geometry>
         <cylinder radius="0.2" length="0.1" />
@@ -69,5 +65,4 @@
     </visual>
     <collision name="left_wheel_collision">
-      <origin xyz="0 0.11 0" rpy="0 1.5707 1.5707"/>
       <geometry>
         <cylinder radius="0.2" length="0.1" />
@@ -76,5 +71,5 @@
     <inertial>
       <mass value="5"/>
-      <origin xyz="0 0 0" rpy="0 1.5707 1.5707"/>
+      <origin xyz="0 0 0" rpy="0 0 0"/>
       <inertia
           ixx="0.1" ixy="0" ixz="0"
@@ -86,5 +81,4 @@
   <link name="right_wheel">
     <visual name="right_wheel_visual">
-      <origin xyz="0 -0.11 0" rpy=" 0 1.5707 1.5707"/>
       <geometry>
         <cylinder radius="0.2" length="0.1" />
@@ -95,5 +89,4 @@
     </visual>
     <collision name="right_wheel_collision">
-      <origin xyz="0 -0.11 0" rpy="0 1.5707 1.5707"/>
       <geometry>
         <cylinder radius="0.2" length="0.1" />
@@ -102,5 +95,5 @@
     <inertial>
       <mass value="5"/>
-      <origin xyz="0 0 0" rpy="0 1.5707 1.5707"/>
+      <origin xyz="0 0 0" rpy="0 0 0"/>
       <inertia
           ixx="0.1" ixy="0" ixz="0"
@@ -110,17 +103,22 @@
     </inertial>
   </link>
+  <joint name="caster_wheel_joint" type="fixed">
+    <parent link="chassis"/>
+    <child link="caster_wheel"/>
+    <origin xyz="0.2 0 -0.1" rpy="0 0 0"/>
+  </joint>
   <joint type="continuous" name="left_wheel_hinge">
-    <origin xyz="0 0.11 0" rpy="0 0 0"/>
+    <origin xyz="-0.2 0.2 0" rpy="-${pi/2} 0 0"/>
     <child link="left_wheel"/>
     <parent link="chassis"/>
-    <axis xyz="0 1 0" rpy="0 0 0"/>
+    <axis xyz="0 0 1"/>
     <limit effort="10000" velocity="1000"/>
     <dynamics damping="1.0" friction="1.0"/>
   </joint>
   <joint type="continuous" name="right_wheel_hinge">
-    <origin xyz="0 -0.11 0" rpy="0 0 0"/>
+    <origin xyz="-0.2 -0.2 0" rpy="${pi/2} 0 0"/>
     <child link="right_wheel"/>
     <parent link="chassis"/>
-    <axis xyz="0 1 0" rpy="0 0 0"/>
+    <axis xyz="0 0 -1"/>
     <limit effort="10000" velocity="1000"/>
     <dynamics damping="1.0" friction="1.0"/>
